Commit message: Fixed mapping simulator stuff

File: SimulationCode/simBotAckermann/urdf/base/base.urdf.xacro (robot description, xacro)
@@ -103,5 +103,5 @@
     <!-- the left Ackermann bar -->
     <joint name="front_left_bar_joint" type="revolute" >
-        <limit lower="-0.5" upper="0.5" effort="100" velocity="10" />
+        <limit lower="-0.9" upper="0.9" effort="100" velocity="10" />
         <axis xyz="0 0 1" />
         <parent link="front_link" />
@@ -131,5 +131,5 @@
     <!-- the right Ackermann bar -->
     <joint name="front_right_bar_joint" type="revolute" >
-        <limit lower="-0.5" upper="0.5" effort="100" velocity="10" />
+        <limit lower="-0.9" upper="0.9" effort="100" velocity="10" />
         <axis xyz="0 0 1" />
         <parent link="front_link" />
@@ -159,5 +159,5 @@
 	<!-- the Ackerman bar -->
     <joint name="ackermann_joint" type="revolute" >
-        <limit lower="-0.5" upper="0.5" effort="100" velocity="10" />
+        <limit lower="-0.9" upper="0.9" effort="100" velocity="10" />
         <axis xyz="0 0 1" />
         <parent link="steer_link" />
@@ -204,5 +204,5 @@
  <!-- a link aligned with the steer direction -->
     <joint name="steer_joint" type="revolute" >
-        <limit lower="-0.5" upper="0.5" effort="100" velocity="10" />
+        <limit lower="-0.9" upper="0.9" effort="100" velocity="10" />
         <axis xyz="0 0 1" />
         <parent link="front_link" />

Commit message: Changed stuff

File: SimulationCode/simBotAckermann/urdf/base/base.urdf.xacro (robot description, xacro)
@@ -103,5 +103,5 @@
     <!-- the left Ackermann bar -->
     <joint name="front_left_bar_joint" type="revolute" >
-        <limit lower="-0.9" upper="0.9" effort="100" velocity="10" />
+        <limit lower="-1.04" upper="1.04" effort="100" velocity="10" />
         <axis xyz="0 0 1" />
         <parent link="front_link" />
@@ -131,5 +131,5 @@
     <!-- the right Ackermann bar -->
     <joint name="front_right_bar_joint" type="revolute" >
-        <limit lower="-0.9" upper="0.9" effort="100" velocity="10" />
+        <limit lower="-1.04" upper="1.04" effort="100" velocity="10" />
         <axis xyz="0 0 1" />
         <parent link="front_link" />
@@ -159,5 +159,5 @@
 	<!-- the Ackerman bar -->
     <joint name="ackermann_joint" type="revolute" >
-        <limit lower="-0.9" upper="0.9" effort="100" velocity="10" />
+        <limit lower="-1.04" upper="1.04" effort="100" velocity="10" />
         <axis xyz="0 0 1" />
         <parent link="steer_link" />
@@ -204,5 +204,5 @@
  <!-- a link aligned with the steer direction -->
     <joint name="steer_joint" type="revolute" >
-        <limit lower="-0.9" upper="0.9" effort="100" velocity="10" />
+        <limit lower="-1.04" upper="1.04" effort="100" velocity="10" />
         <axis xyz="0 0 1" />
         <parent link="front_link" />
